File: efi-shield-rev01.sch (EAGLE design)
At the start: 6 parts

Commit message: Connection sheet done + added all sheets.
Parts:
- added J7: AMPSEAL-23POS-HEADER, cpsmv:AMPSEAL-23POS-HEADER
- added SPI: (no value), pinhead:PINHD-2X3
- J1: value (none) -> PWMH; device cpsmv:PINHD-1X8 -> cpsmv:PINHD-1X10
- J2: value (none) -> PWMI
- J3: value (none) -> COMM
- J4: value (none) -> PWR
- J5: value (none) -> ADCL
- J6: value (none) -> ADCH; device cpsmv:PINHD-1X10 -> cpsmv:PINHD-1X8
Connections:
- new net +12V: J4.8
- new net +3V3: J4.2, J4.4
- new net +5V: J4.5, SPI.2
- new net CS1_3V3: J2.4
- new net ECT_3V3: J6.1
- new net FUEL: J1.10
- new net GND: J1.4, J4.6, J4.7, SPI.6
- new net HALL: J2.3
- new net IAT_3V3: J5.8
- new net MAP_DIV: J5.1
- new net MISO_3V3: SPI.1
- new net MOSI_3V3: SPI.4
- new net O2_DIV: J5.2
- new net RESET: SPI.5
- new net SCK_3V3: SPI.3
- new net SPARK: J2.1
- new net TPS: J6.4
Other:
- note added: "A0 A1 A2 A3 A4 A5 A6 A7"
- note added: "A8 A9 A10 A11 DAC0 DAC1 CANRX CANTX"
- note added: "AMPSEAL"
- note added: "ARDUINO DUE"
- note added: "D14/TX3 D15/RX3 D16/TX2 D17/RX2 D18/TX1 D19/RX1 D20/SDA D21/SCL"
- note added: "D7 D6 D5 D4/SD-CS D3 D2 D1/TX0 D0/RX0"
- note added: "NC IOREF RESET 3.3V 5V GND GND VIN"
- note added: "SCL1 SDA1 AREF GND D13 D12 D11 D10/ETH-CS D9 D8"
- note added: "SPI"
