File: efi-shield.brd (EAGLE design)
At the start: 117.5 x 78 mm, 174 parts, among them J1 PWMH, J10 MOLEX-85505-5002, J2 PWMI, J3 COMM, J4 PWR, J5 ADCL, J6 ADCH, J7 AMPSEAL-23POS-HEADER, J8 SPI, J9 MOLEX-85505-5002, Q1 PN2222A, Q2 FJPF13009, Q3 PN2222A, Q4 PN2222A, Q5 PN2222A, Q6 PN2222A, Q7 ISL9V5036P3_F085, SW1 CTS-204-211ST, U1 TXS0104E, U10 MCP2551-I/SN, U2 TXS0104E, U3 MCP3304, U4 MCP6024, U5 MCP6024, U6 MCP6022, U7 NE555DR, U8 MCP4142-104, U9 MCP4142-103

Commit message: Low-impedance termination tach circuitadded. Removed one-shot/digi-pot and LPF tach circuit.
Parts:
- removed C26, C27: 330pF, cpsmv:C050-025X075
- removed C28, C29: 10nF, cpsmv:C050-025X075
- removed C30, C31, C32: 0.1uF, cpsmv:C050-025X075
- removed R18, R19: 100kΩ, cpsmv:0207/7
- removed R45: 0Ω, cpsmv:0207/7
- removed TP40: HALL, cpsmv:TP-P1-20
- removed TP41: HALL_FIL, cpsmv:TP-P1-20
- removed TP42: TACH_5V, cpsmv:TP-P1-20
- removed TP43: TACH_3V3, cpsmv:TP-P1-20
- removed U6: MCP6022, cpsmv:SOIC127P600X175-8N
- removed U7: NE555DR, cpsmv:SOIC127P600X175-8N
- removed U8: MCP4142-104, cpsmv:DIP254P762X533-8
- removed U9: MCP4142-103, cpsmv:DIP254P762X533-8
- C25: value 47nF -> 68nF
- R20: value 36kΩ -> 220Ω
- R21: value 64kΩ -> 390Ω
- moved R21 379.1 mm to (80.5, 317.4)
- moved R20 366.1 mm to (80.5, 321.7)
- moved C25 305.7 mm to (79.0, 312.7)
Connections:
- removed net HALL_FIL: C26.1, R45.1, TP41.TP, U6.1, U6.2
- removed net N$13: C27.1, R19.2, U6.3
- removed net N$22: C26.2, R18.2, R19.1
- removed net N$23: U8.6, U9.5
- removed net N$24: C29.1, U7.5
- removed net N$4: C32.1, U7.6, U7.7, U9.6
- removed net N$45: R45.2, U7.2
- removed net TACH_3V3: J2.3, R20.2, R21.2, TP43.TP
- removed net TACH_5V: R20.1, TP42.TP, U7.3
- net +5V: now also R20.2; no longer C25.1, C28.1, C30.1, C31.1, U6.8, U7.4, U7.8, U8.5, U8.8, U9.8
- net AGND: no longer C25.2, C27.2, U6.4
- net CS2_5V: no longer U8.1
- net CS3_5V: no longer U9.1
- net GND: now also C25.2; no longer C28.2, C29.2, C30.2, C31.2, C32.2, U7.1, U8.4, U9.4
- net HALL: now also C25.1, J2.3, R20.1, R21.2; no longer R18.1, TP40.TP
- net MISO_5V: no longer U8.7, U9.7
- net MOSI_5V: no longer U8.3, U9.3
- net SCK_5V: no longer U8.2, U9.2

Commit message: Changed analog input filters + tach circuit.
Parts:
- removed C10, C11, C12, C20, C21, C22, C9: 330pF, cpsmv:C050-025X075
- removed C23: 2.2uF, cpsmv:C050-025X075
- removed C24: 0.1uF, cpsmv:C050-025X075
- removed C25: 68nF, cpsmv:C050-025X075
- removed JP4: SPR_A1, cpsmv:1X01
- removed JP5: SPR_A2, cpsmv:1X01
- removed JP6: SPR_A3, cpsmv:1X01
- removed R39, R40, R41, R42, R43, R44: 0Ω, cpsmv:0207/7
- removed TP14: CS3_3V3, cpsmv:TP-P1-20
- removed TP15: CS2_3V3, cpsmv:TP-P1-20
- removed TP20: MAP, cpsmv:TP-P1-20
- removed TP21: MAP_FIL, cpsmv:TP-P1-20
- removed TP22: TPS, cpsmv:TP-P1-20
- removed TP23: TPS_FIL, cpsmv:TP-P1-20
- removed TP24: IAT, cpsmv:TP-P1-20
- removed TP25: IAT_FIL, cpsmv:TP-P1-20
- removed TP26: ECT, cpsmv:TP-P1-20
- removed TP27: ECT_FIL, cpsmv:TP-P1-20
- removed TP28: O2, cpsmv:TP-P1-20
- removed TP29: O2_FIL, cpsmv:TP-P1-20
- removed TP30: SPR_A1, cpsmv:TP-P1-20
- removed TP31: SPR_A1_FIL, cpsmv:TP-P1-20
- removed TP32: SPR_A2, cpsmv:TP-P1-20
- removed TP33: SPR_A2_FIL, cpsmv:TP-P1-20
- removed TP34: SPR_A3, cpsmv:TP-P1-20
- removed TP35: SPR_A3_FIL, cpsmv:TP-P1-20
- removed TP52: CS2_5V, cpsmv:TP-P1-20
- removed TP53: CS3_5V, cpsmv:TP-P1-20
- removed U3: MCP3304, cpsmv:SOIC127P600X175-16N
- removed U4: MCP6024, cpsmv:SOIC127P600X175-14N
- added R18, R71, R74, R80, R83, R89: 120kΩ, cpsmv:0207/7
- added R19, R72, R81, R90: 56kΩ, cpsmv:0207/7
- added R64: 220Ω, cpsmv:0207/7
- added R65: 390Ω, cpsmv:0207/7
- added R66, R75, R84: 68kΩ, cpsmv:0207/7
- added R67, R76, R85: 3.9kΩ, cpsmv:0207/7
- added R68, R77, R86: 39kΩ, cpsmv:0207/7
- added R69, R70, R78, R79, R87, R88: 82kΩ, cpsmv:0207/7
- added R73, R82: 180kΩ, cpsmv:0207/7
- added U7, U8, U9: LM358, cpsmv:SOP08
- C13: value 330pF -> 6.8nF
- C14, C5: value 47nF -> 10nF
- C16, C18: value 330pF -> 10nF
- C3: value 0.1uF -> 10nF
- C4: value 0.1uF -> 47nF
- C6: value 330pF -> 47nF
- R10: value 100kΩ -> 56kΩ
- R11, R2: value 100kΩ -> 180kΩ
- R12, R3, R9: value 100kΩ -> 120kΩ
- R13, R4: value 100kΩ -> 68kΩ
- R14, R5: value 100kΩ -> 3.9kΩ
- R15, R6: value 100kΩ -> 39kΩ
- R16, R17, R7, R8: value 100kΩ -> 330kΩ
- R20: value 220Ω -> 180kΩ
- R21: value 390Ω -> 120kΩ
- R37, R38: value 0Ω -> 680Ω
- U2: value TXS0104E -> LM358; device cpsmv:SOIC127P600X175-14N -> cpsmv:SOP08
- U5: value MCP6024 -> LM358; device cpsmv:SOIC127P600X175-14N -> cpsmv:SOP08
- moved R20 791.3 mm to (-373.4, -326.5)
- moved R21 781.0 mm to (-361.6, -326.5)
- moved R38 650.5 mm to (-373.4, -369.7)
- moved R37 650.2 mm to (-373.4, -365.4)
- moved C15 643.8 mm to (-374.9, -321.7)
- moved C16 637.5 mm to (-366.4, -321.7)
- moved C8 636.1 mm to (-374.9, -379.6)
- moved C7 632.6 mm to (-374.9, -374.4)
- moved C17 631.7 mm to (-357.9, -321.7)
- moved C18 626.3 mm to (-349.4, -321.7)
- moved C19 621.3 mm to (-340.9, -321.7)
- moved R12 573.3 mm to (-373.4, -190.2)
- moved R6 571.8 mm to (-373.4, -155.3)
- moved R7 569.9 mm to (-373.4, -159.6)
- moved R11 569.8 mm to (-364.9, -185.0)
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Connections:
- removed net CS2_3V3: TP15.TP, U2.2
- removed net CS2_5V: TP52.TP, U2.13
- removed net CS3_3V3: TP14.TP, U2.3
- removed net CS3_5V: TP53.TP, U2.12
- removed net ECT_ADC: R40.2, U3.4
- removed net IAT_ADC: R39.2, U3.3
- removed net MAP_ADC: R37.2, U3.1
- removed net N$15: C15.2, R10.2, R11.1
- removed net N$16: C18.1, R13.2, U5.5
- removed net N$17: C17.2, R12.2, R13.1
- removed net N$18: C20.1, R15.2, U5.10
- removed net N$19: C19.2, R14.2, R15.1
- removed net N$20: C22.1, R17.2, U5.12
- removed net N$21: C21.2, R16.2, R17.1
- removed net O2_ADC: R41.2, U3.5
- removed net SPRA1ADC: R42.2, U3.6
- removed net SPRA2ADC: R43.2, U3.7
- removed net SPRA3ADC: R44.2, U3.8
- removed net SPR_A1: JP4.1, R12.1, TP30.TP
- removed net SPR_A1_FIL: C17.1, R42.1, TP31.TP, U5.6, U5.7
- removed net SPR_A2: JP5.1, R14.1, TP32.TP
- removed net SPR_A2_FIL: C19.1, R43.1, TP33.TP, U5.8, U5.9
- removed net SPR_A3: JP6.1, R16.1, TP34.TP
- removed net SPR_A3_FIL: C21.1, R44.1, TP35.TP, U5.13, U5.14
- removed net TPS_ADC: R38.2, U3.2
- new net N$13: C6.1, R16.2, R17.2, U2.6
- new net N$4: R10.2, R9.2, U5.5
- new net N$53: R66.2, R67.2, U7.3
- new net N$54: R71.2, R72.2, U7.5
- new net N$55: R20.2, R21.2, U7.2
- new net N$56: R21.1, R69.1, U7.1
- new net N$57: C15.1, R69.2, R70.2, U7.6
- new net N$58: R67.1, R68.2
- new net N$59: R75.2, R76.2, U8.3
- new net N$60: R80.2, R81.2, U8.5
- new net N$61: R73.2, R74.2, U8.2
- new net N$62: R74.1, R78.1, U8.1
- new net N$63: C17.1, R78.2, R79.2, U8.6
- new net N$64: R76.1, R77.2
- new net N$65: R84.2, R85.2, U9.3
- new net N$66: R89.2, R90.2, U9.5
- new net N$67: R82.2, R83.2, U9.2
- new net N$68: R83.1, R87.1, U9.1
- new net N$69: C19.1, R87.2, R88.2, U9.6
- new net N$70: R85.1, R86.2
- net +3V3: no longer C4.1, U2.1
- net +5V: now also C16.1, C18.1, R13.1, R18.1, R37.2, R38.2, R4.1, R64.2, R66.1, R71.1, R75.1, R80.1, R84.1, R89.1, R9.1, U2.8, U5.8, U7.8, U8.8, U9.8; no longer C23.1, C24.1, R20.2, U2.14, U3.15, U3.16, U4.4, U5.4
- net AGND: no longer C11.2, C13.2, C14.2, C16.2, C18.2, C20.2, C22.2, C23.2, C24.2, C5.2, C7.2, C9.2, U3.14, U3.9, U4.11, U5.11
- net CS1_5V: no longer U3.10
- net ECT: now also C7.1, R2.1, R37.1; no longer R8.1, TP26.TP
- net ECT_FIL: now also C4.2, R8.1, U5.7; no longer C12.1, R40.1, TP27.TP, U4.13, U4.14
- net GND: now also C13.2, C14.2, C16.2, C18.2, C5.2, C7.2, C8.2, R10.1, R15.1, R19.1, R6.1, R65.1, R68.1, R72.1, R77.1, R81.1, R86.1, R90.1, U2.4, U5.4, U7.4, U8.4, U9.4; no longer C25.2, C4.2, R21.1, U2.7
- net HALL: now also C13.1, R64.1, R65.2; no longer C25.1, R20.1, R21.2
- net IAT: now also C8.1, R11.1, R38.1; no longer R6.1, TP24.TP
- net IAT_FIL: now also C6.2, R17.1, U2.7; no longer C10.1, R39.1, TP25.TP, U4.8, U4.9
- net MAP: now also R20.1; no longer R2.1, TP20.TP
- net MAP_FIL: now also C15.2, R70.1, U7.7; no longer C6.1, R37.1, TP21.TP, U4.1, U4.2
- net MISO_5V: no longer U3.12
- net MOSI_5V: no longer U3.11
- net N$10: now also R18.2, R19.2, U2.5; no longer C13.1, R9.2, U4.12
- net N$11: now also R11.2, R12.2, U2.2; no longer C12.2, R8.2, R9.1
- net N$12: now also R12.1, R16.1, U2.1; no longer U2.8
- net N$14: now also R14.1, R15.2; no longer C16.1, R11.2, U5.3
- net N$2: now also R4.2, R5.2, U5.3; no longer C7.1, R3.2, U4.3
- net N$5: now also R3.2, U5.2; no longer C6.2, R3.1
- net N$6: now also R3.1, R7.1, U5.1; no longer C9.1, R5.2, U4.5
- net N$7: now also C4.1, R7.2, R8.2, U5.6; no longer C8.2, R4.2, R5.1
- net N$8: now also R13.2, R14.2, U2.3; no longer C11.1, R7.2, U4.10
- net N$9: now also R5.1; no longer C10.2, R7.1
- net O2: now also R73.1; no longer R10.1, TP28.TP
- net O2_FIL: now also C17.2, R79.1, U8.7; no longer C15.1, R41.1, TP29.TP, U5.1, U5.2
- net SCK_5V: no longer U3.13
- net TPS: now also R82.1; no longer R4.1, TP22.TP
- net TPS_FIL: now also C19.2, R88.1, U9.7; no longer C8.1, R38.1, TP23.TP, U4.6, U4.7

Commit message: New test points, high frequency blocker for MAP, killswitch voltage divider.
Parts:
- removed TP9: AGND, cpsmv:TP-P1-20
- added C10: 220pF, cpsmv:C050-025X075
- added C9: 330pF, cpsmv:C050-025X075
- added R39: 470Ω, cpsmv:0207/7
- added R40: 1kΩ, cpsmv:0207/7
- added R41: 2.7kΩ, cpsmv:0207/7
- added TP14: HALL, cpsmv:TP-P1-20
- added TP15: ECT, cpsmv:TP-P1-20
- added TP20: ECT_FIL, cpsmv:TP-P1-20
- added TP21: IAT, cpsmv:TP-P1-20
- added TP22: IAT_FIL, cpsmv:TP-P1-20
- added TP23: MAP, cpsmv:TP-P1-20
- added TP24: MAP_FIL, cpsmv:TP-P1-20
- added TP25: O2, cpsmv:TP-P1-20
- added TP26: O2_FIL, cpsmv:TP-P1-20
- added TP27: TPS, cpsmv:TP-P1-20
- added TP28: TPS_FIL, cpsmv:TP-P1-20
- TP7: value AGND -> KILL_SW
- TP8: value AGND -> KILL_SW_3V3
- moved TP8 632.9 mm to (-461.5, -401.2), turned to 0 degrees
- moved TP7 618.9 mm to (-455.0, -401.2), turned to 0 degrees
Connections:
- removed net AGND: TP7.TP, TP8.TP, TP9.TP
- new net KILL_SW: R40.1, TP7.TP
- new net KILL_SW_3V3: C10.1, R40.2, R41.2, TP8.TP
- net ECT: now also TP15.TP
- net ECT_FIL: now also TP20.TP
- net GND: now also C10.2, C9.2, R39.1, R41.1
- net HALL: now also TP14.TP
- net IAT: now also TP21.TP
- net IAT_FIL: now also TP22.TP
- net MAP: now also C9.1, R39.2, TP23.TP
- net MAP_FIL: now also TP24.TP
- net O2: now also TP25.TP
- net O2_FIL: now also TP26.TP
- net TPS: now also TP27.TP
- net TPS_FIL: now also TP28.TP
